File: 820.kicad_pcb (KiCad board)
At the start: 4 copper layers, 48 x 105 mm, 124 parts, among them J1 PJ301BM, J10 PJ301BM, J2 PJ301BM, J4 PJ301BM, J5 PJ301BM, J6 PJ301BM, J7 PJ301BM, J8 PJ301BM, J9 PJ301BM, P1 CONN_02X05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

Commit message: first commit in a while. switched matched pair to PMP and other stuff. getting ready to order r1.1
Parts:
- added R14: 16.9R, MyModules:SM0603-R-YAGEO, B.Cu at (120.2, 81.6)
- TC1: value 1K 3300ppm/K -> 500R ±3850ppm/°C; footprint MyModules:SM0603-R-YAGEO -> Resistors_SMD:R_0805
- moved C1 4.56 mm to (123.7, 77.5)
- moved TC1 0.94 mm to (117.2, 81.6)
- moved Q1 0.64 mm to (117.2, 83.8), turned to 0 degrees
- moved R17 0.11 mm to (113.6, 80.8)
Connections:
- TC1 pad 2: GND -> Net-(R14-Pad2)
Routing:
- net Net-(Q1-Pad6): track 10.2 -> 7.40 mm
- net +12V: track 217.7 -> 220.0 mm
- net Net-(Q1-Pad2): track 3.90 -> 5.44 mm
- net Net-(R14-Pad2): track 0.00 -> 1.20 mm
- net Net-(Q1-Pad4): track 3.15 -> 2.27 mm
